Commit message: update in xacro

File: omnibase_description/xacro/rim.urdf.xacro (robot description, xacro)
@@ -1,9 +1,6 @@
 <?xml version="1.0" ?>
 <robot xmlns:xacro="http://www.ros.org/wiki/xacro">
-	<xacro:include filename="$(find open_base)/xacro/roller.urdf.xacro"/>
-	<xacro:macro
-		name="rim_macro"
-		params="name color xyz rpy"
-	>
+	<xacro:include filename="$(find omnibase_description)/xacro/roller.urdf.xacro"/>
+	<xacro:macro name="rim_macro" params="name color xyz rpy">
 		<link name="rim_${name}_link">
 			<inertial>
@@ -21,5 +18,5 @@
 			<visual>
 				<geometry>
-					<mesh filename="package://open_base/mesh/rim.stl"/>
+					<mesh filename="package://omnibase_description/meshes/rim.stl"/>
 				</geometry>
 				<material name="rim_${name}_material">
@@ -29,12 +26,9 @@
 			<collision>
 				<geometry>
-					<mesh filename="package://open_base/mesh/rim.stl"/>
+					<mesh filename="package://omnibase_description/meshes/rim.stl"/>
 				</geometry>
 			</collision>
 		</link>
-		<joint
-			name="rim_${name}_joint"
-			type="continuous"
-		>
+		<joint name="rim_${name}_joint" type="continuous">
 			<parent link="base_link" />
 			<child link="rim_${name}_link" />

File: omnibase_description/xacro/roller.urdf.xacro (robot description, xacro)
@@ -1,8 +1,5 @@
 <?xml version="1.0" ?>
 <robot xmlns:xacro="http://www.ros.org/wiki/xacro">
-	<xacro:macro
-		name="roller_macro"
-		params="parent name xyz rpy"
-	>
+	<xacro:macro name="roller_macro" params="parent name xyz rpy">
 		<link name="roller_${name}_rim_${parent}_link">
 			<inertial>
@@ -19,5 +16,5 @@
 			<visual>
 				<geometry>
-					<mesh filename="package://open_base/mesh/roller.stl"/>
+					<mesh filename="package://omnibase_description/meshes/roller.stl"/>
 				</geometry>
 				<material name="roller_material">
@@ -27,19 +24,16 @@
 			<collision>
 				<geometry>
-					<mesh filename="package://open_base/mesh/roller.stl"/>
+					<mesh filename="package://omnibase_description/meshes/roller.stl"/>
 				</geometry>
 			</collision>
 		</link>
-		<joint
-			name="roller_${name}_rim_${parent}_joint"
-			type="continuous"
-		>
+		<gazebo reference="base_link">
+    		<material>Gazebo/White</material>
+  		</gazebo>
+		<joint name="roller_${name}_rim_${parent}_joint" type="continuous">
 			<parent link="rim_${parent}_link"/>
 			<child link="roller_${name}_rim_${parent}_link"/>
 			<axis xyz="0 0 1"/>
-			<origin
-				xyz="${xyz}"
-				rpy="${rpy}"
-			/>
+			<origin xyz="${xyz}" rpy="${rpy}"/>
 		</joint>
 	</xacro:macro>

Commit message: Changed to JointVelocityController

File: omnibase_description/xacro/rim.urdf.xacro (robot description, xacro)
@@ -90,8 +90,8 @@
 			<type>transmission_interface/SimpleTransmission</type>
 			<joint name="rim_${name}_joint">
-				<hardwareInterface>hardware_interface/EffortJointInterface</hardwareInterface>
+				<hardwareInterface>hardware_interface/VelocityJointInterface</hardwareInterface>
 			</joint>
 			<actuator name="rim_${name}_motor">
-				<hardwareInterface>hardware_interface/EffortJointInterface</hardwareInterface>
+				<hardwareInterface>hardware_interface/VelocityJointInterface</hardwareInterface>
 				<mechanicalReduction>1</mechanicalReduction>
 			</actuator>

File: omnibase_description/xacro/roller.urdf.xacro (robot description, xacro)
@@ -22,9 +22,9 @@
 				</material>
 			</visual>
-			<collision>
+			<!-- <collision>
 				<geometry>
 					<mesh filename="package://omnibase_description/meshes/roller.stl"/>
 				</geometry>
-			</collision>
+			</collision> -->
 		</link>
 		<gazebo reference="base_link">
