Commit message: wheel size small for easy viewing

File: omnibase_description/xacro/wheel.urdf.xacro (robot description, xacro)
@@ -11,5 +11,5 @@
 				<origin xyz="0 0 0" rpy="0 0 0" />
 				<geometry>
-					<cylinder length="0.02" radius="0.04" />
+					<cylinder length="0.01" radius="0.01" />
 				</geometry>
 			</visual>
@@ -17,5 +17,5 @@
 				<origin xyz="0 0 0" rpy="0 0 0" />
 				<geometry>
-					<cylinder length="0.02" radius="0.04" />
+					<cylinder length="0.01" radius="0.01" />
 				</geometry>
 				<surface>
