Commit message: model update

File: omnibase_description/xacro/gazebo.urdf.xacro (robot description, xacro)
@@ -55,3 +55,11 @@
     </sensor>
   </gazebo>
+  <gazebo>
+    <plugin name="ground_truth" filename="libgazebo_ros_p3d.so">
+      <frameName>world</frameName>
+      <bodyName>base_link</bodyName>
+      <topicName>odom</topicName>
+      <updateRate>30.0</updateRate>
+    </plugin>
+  </gazebo>
 </robot>

File: omnibase_description/xacro/main.urdf.xacro (robot description, xacro)
@@ -32,26 +32,26 @@
 		<parent link="origin_link" />
 		<child link="base_link" />
-		<origin xyz="0 0 0"/>
+		<origin xyz="0 0 0.05"/>
 	</joint>
 	<xacro:rim_macro
 		name="front_right"
 		color="0.3 0 0"
-		xyz="0.053181445 0.052283625 0"
-		rpy="1.570796326794896 0 -0.73"/>
+		xyz="0.053 0.05300221419 0"
+		rpy="1.570796326794896 0 -0.81"/>
 	<xacro:rim_macro
 		name="back_right"
 		color="0 0 0.3"
-		xyz="0.053181445 -0.052283625 0"
-		rpy="1.570796326794896 0 -2.42"/>
+		xyz="0.053 -0.05300221419 0"
+		rpy="1.570796326794896 0 -2.39"/>
 	<xacro:rim_macro
 		name="back_left"
 		color="0 0.3 0"
-		xyz="-0.053181445 -0.052283625 0"
-		rpy="1.570796326794896 0 2.42"/>
+		xyz="-0.053 -0.05300221419 0"
+		rpy="1.570796326794896 0 2.39"/>
 	<xacro:rim_macro
 		name="front_left"
 		color="0 0.2 0.2"
-		xyz="-0.053181445 0.052283625 0"
-		rpy="1.570796326794896 0 0.73"/>
+		xyz="-0.053 0.05300221419 0"
+		rpy="1.570796326794896 0 0.81"/>
 	<joint name="scan_joint" type="fixed">
     	<parent link="base_link"/>

Commit message: model changes and readme update

File: omnibase_description/xacro/gazebo.urdf.xacro (robot description, xacro)
@@ -6,14 +6,14 @@
         <material>Gazebo/White</material>
     </gazebo>
-    <gazebo reference="rim_front_right_link">
+    <gazebo reference="rim_front_left_link">
         <material>Gazebo/Red</material>
     </gazebo>
-  <gazebo reference="rim_back_right_link">
+  <gazebo reference="rim_front_right_link">
         <material>Gazebo/Green</material>
     </gazebo>
-    <gazebo reference="rim_back_left_link">
+    <gazebo reference="rim_back_right_link">
         <material>Gazebo/Blue</material>
     </gazebo>
-  <gazebo reference="rim_front_left_link">
+  <gazebo reference="rim_back_left_link">
         <material>Gazebo/Yellow</material>
     </gazebo>

File: omnibase_description/xacro/main.urdf.xacro (robot description, xacro)
@@ -32,23 +32,23 @@
 		<parent link="origin_link" />
 		<child link="base_link" />
-		<origin xyz="0 0 0.05"/>
+		<origin xyz="0 0 0.02"/>
 	</joint>
 	<xacro:rim_macro
-		name="front_right"
+		name="front_left"
 		color="0.3 0 0"
 		xyz="0.053 0.05300221419 0"
 		rpy="1.570796326794896 0 -0.81"/>
 	<xacro:rim_macro
-		name="back_right"
+		name="front_right"
 		color="0 0 0.3"
 		xyz="0.053 -0.05300221419 0"
 		rpy="1.570796326794896 0 -2.39"/>
 	<xacro:rim_macro
-		name="back_left"
+		name="back_right"
 		color="0 0.3 0"
 		xyz="-0.053 -0.05300221419 0"
 		rpy="1.570796326794896 0 2.39"/>
 	<xacro:rim_macro
-		name="front_left"
+		name="back_left"
 		color="0 0.2 0.2"
 		xyz="-0.053 0.05300221419 0"
@@ -57,5 +57,5 @@
     	<parent link="base_link"/>
     	<child link="base_scan"/>
-    	<origin xyz="-0.032 0 0.072" rpy="0 0 0"/>
+    	<origin xyz="-0.005 0 0.064" rpy="0 0 0"/>
   	</joint>
 	<link name="base_scan">
@@ -63,5 +63,5 @@
     	<origin xyz="0 0 0.0" rpy="0 0 0"/>
     	<geometry>
-       		<mesh filename="package://omnibase_description/meshes/lds.stl" scale="0.0004 0.0004 0.0004"/>
+       		<mesh filename="package://omnibase_description/meshes/lds.stl" scale="0.0003 0.0003 0.0003"/>
       	</geometry>
       	<material name="dark"/>
@@ -80,4 +80,24 @@
                izz="0.001" />
     </inertial>
-  </link>
+  	</link>
+  	<joint name="body_joint" type="fixed">
+  		<parent link="base_link"/>
+  		<child link="body_link"/>
+  		<origin xyz="0 0 0.03" rpy="1.57 0 3.14"/>
+  	</joint>
+  	<link name="body_link">
+  		<visual>
+  			<geometry>
+       			<mesh filename="package://omnibase_description/meshes/body.STL"/>
+      		</geometry>
+      		<material name="base_material"/>
+      	</visual>
+      	<inertial>
+      		<mass value="0.1" />
+      		<origin xyz="0 0 0" />
+      		<inertia 	ixx="0.000056443" ixy="0.0" ixz="0.0"
+               			iyy="0.0012923047" iyz="0.0"
+               			izz="0.000113232" />
+    	</inertial>
+  	</link>
 </robot>

Commit message: Added textures

File: omnibase_description/xacro/gazebo.urdf.xacro (robot description, xacro)
@@ -3,17 +3,20 @@
   <xacro:arg name="laser_visual" default="false"/>
   <xacro:arg name="imu_visual"   default="false"/>
-  <gazebo reference="base_link">
+  <!-- <gazebo reference="base_link">
         <material>Gazebo/White</material>
-    </gazebo>
-    <gazebo reference="rim_front_left_link">
+    </gazebo> -->
+    <!-- <gazebo reference="base_link">
+			<material>Gazebo/Yellow</material>
+		</gazebo> -->
+    <gazebo reference="front_left_wheel_link">
         <material>Gazebo/Red</material>
     </gazebo>
-  <gazebo reference="rim_front_right_link">
+  <gazebo reference="front_right_wheel_link">
         <material>Gazebo/Green</material>
     </gazebo>
-    <gazebo reference="rim_back_right_link">
+    <gazebo reference="back_right_wheel_link">
         <material>Gazebo/Blue</material>
     </gazebo>
-  <gazebo reference="rim_back_left_link">
+  <gazebo reference="back_left_wheel_link">
         <material>Gazebo/Yellow</material>
     </gazebo>

File: omnibase_description/xacro/main.urdf.xacro (robot description, xacro)
@@ -18,13 +18,10 @@
 	<visual>
 		<geometry>
-			<mesh filename="package://omnibase_description/meshes/trotbot_full_stl.stl" scale="0.001 0.001 0.001"/>
+			<mesh filename="package://omnibase_description/meshes/trotbot.dae" />
 		</geometry>
-		<material name="base_material">
-			<color rgba="1 1 1 1"/>
-		</material>
 	</visual>
 	<collision>
 		<geometry>
-			<mesh filename="package://omnibase_description/meshes/trotbot_full_stl.stl" scale="0.001 0.001 0.001"/>
+			<mesh filename="package://omnibase_description/meshes/trotbot.dae" />
 		</geometry>
 	</collision>
