Commit message: added launch files

File: omnibase_description/xacro/main.urdf.xacro (robot description, xacro)
@@ -16,5 +16,5 @@
 	<visual>
 		<geometry>
-			<mesh filename="package://omnibase_description/meshes/new_base.stl"/>
+			<mesh filename="package://omnibase_description/meshes/sq_base.stl"/>
 		</geometry>
 		<material name="base_material">
@@ -24,5 +24,5 @@
 	<collision>
 		<geometry>
-			<mesh filename="package://omnibase_description/meshes/new_base.stl"/>
+			<mesh filename="package://omnibase_description/meshes/sq_base.stl"/>
 		</geometry>
 	</collision>
@@ -34,25 +34,37 @@
 	</joint>
 	<xacro:rim_macro
-		name="front_left"
+		name="front_right"
 		color="0.3 0 0"
-		xyz="-0.05 0.05 0"
-		rpy="1.570796326794896 0 1.047197551196597"/>
+		xyz="0.053181445 0.052283625 0"
+		rpy="1.570796326794896 0 -0.73"/>
 	<xacro:rim_macro
 		name="back_right"
-		color="0 0.3 0"
-		xyz="0.05 -0.05 0"
-		rpy="1.570796326794896 0 3.141592653589793"/>
-	<xacro:rim_macro
-		name="front_right"
 		color="0 0 0.3"
-		xyz="0.05 0.05 0"
-		rpy="1.570796326794896 0 -1.047197551196597"/>
+		xyz="0.053181445 -0.052283625 0"
+		rpy="1.570796326794896 0 -2.42"/>
 	<xacro:rim_macro
 		name="back_left"
-		color="0 0 0.3"
-		xyz="-0.05 -0.05 0"
-		rpy="1.570796326794896 0 -1.047197551196597"/>
+		color="0 0.3 0"
+		xyz="-0.053181445 -0.052283625 0"
+		rpy="1.570796326794896 0 2.42"/>
+	<xacro:rim_macro
+		name="front_left"
+		color="0 0.2 0.2"
+		xyz="-0.053181445 0.052283625 0"
+		rpy="1.570796326794896 0 0.73"/>
 	<gazebo reference="base_link">
     		<material>Gazebo/White</material>
+  	</gazebo>
+  	<gazebo reference="rim_front_right_link">
+    		<material>Gazebo/Red</material>
+  	</gazebo>
+	<gazebo reference="rim_back_right_link">
+    		<material>Gazebo/Green</material>
+  	</gazebo>
+  	<gazebo reference="rim_back_left_link">
+    		<material>Gazebo/Blue</material>
+  	</gazebo>
+	<gazebo reference="rim_front_left_link">
+    		<material>Gazebo/Yellow</material>
   	</gazebo>
   	<gazebo>

Commit message: added gazebo xacro and lidar

File: omnibase_description/xacro/main.urdf.xacro (robot description, xacro)
@@ -2,4 +2,5 @@
 <robot xmlns:xacro="http://www.ros.org/wiki/xacro" name="omnibase">
 	<xacro:include filename="$(find omnibase_description)/xacro/rim.urdf.xacro"/>
+	<xacro:include filename="$(find omnibase_description)/xacro/gazebo.urdf.xacro"/>
 	<link name="origin_link"/>
 	<link name="base_link">
@@ -53,23 +54,30 @@
 		xyz="-0.053181445 0.052283625 0"
 		rpy="1.570796326794896 0 0.73"/>
-	<gazebo reference="base_link">
-    		<material>Gazebo/White</material>
-  	</gazebo>
-  	<gazebo reference="rim_front_right_link">
-    		<material>Gazebo/Red</material>
-  	</gazebo>
-	<gazebo reference="rim_back_right_link">
-    		<material>Gazebo/Green</material>
-  	</gazebo>
-  	<gazebo reference="rim_back_left_link">
-    		<material>Gazebo/Blue</material>
-  	</gazebo>
-	<gazebo reference="rim_front_left_link">
-    		<material>Gazebo/Yellow</material>
-  	</gazebo>
-  	<gazebo>
-		<plugin name="gazebo_ros_control" filename="libgazebo_ros_control.so">
-		<robotNamespace>omnibase</robotNamespace>
-		</plugin>
-	</gazebo>
+	<joint name="scan_joint" type="fixed">
+    	<parent link="base_link"/>
+    	<child link="base_scan"/>
+    	<origin xyz="-0.032 0 0.072" rpy="0 0 0"/>
+  	</joint>
+	<link name="base_scan">
+    <visual>
+    	<origin xyz="0 0 0.0" rpy="0 0 0"/>
+    	<geometry>
+       		<mesh filename="package://omnibase_description/meshes/lds.stl" scale="0.0004 0.0004 0.0004"/>
+      	</geometry>
+      	<material name="dark"/>
+    </visual>
+    <!-- <collision>
+      <origin xyz="0.015 0 -0.0065" rpy="0 0 0"/>
+      <geometry>
+        <cylinder length="0.0315" radius="0.055"/>
+      </geometry>
+    </collision> -->
+    <inertial>
+      <mass value="0.114" />
+      <origin xyz="0 0 0" />
+      <inertia ixx="0.001" ixy="0.0" ixz="0.0"
+               iyy="0.001" iyz="0.0"
+               izz="0.001" />
+    </inertial>
+  </link>
 </robot>

Commit message: fixed xacro

File: omnibase_description/xacro/main.urdf.xacro (robot description, xacro)
@@ -32,5 +32,5 @@
 		<parent link="origin_link" />
 		<child link="base_link" />
-		<origin xyz="0 0 0.05"/>
+		<origin xyz="0 0 0"/>
 	</joint>
 	<xacro:rim_macro

Commit message: Added Husky Wheel Ref

File: omnibase_description/xacro/main.urdf.xacro (robot description, xacro)
@@ -38,5 +38,7 @@
 		color="0.3 0 0"
 		xyz="0.053 0.05300221419 0"
-		rpy="1.570796326794896 0 -0.81"/>
+		rpy="1.570796326794896 0 -0.81">
+	<mesh scale="10 10 10"/>
+	</xacro:rim_macro>
 	<xacro:rim_macro
 		name="front_right"

Commit message: Added coeff of restitution

File: omnibase_description/xacro/main.urdf.xacro (robot description, xacro)
@@ -3,4 +3,5 @@
 	<xacro:include filename="$(find omnibase_description)/xacro/rim.urdf.xacro"/>
 	<xacro:include filename="$(find omnibase_description)/xacro/gazebo.urdf.xacro"/>
+	<xacro:include filename="$(find omnibase_description)/xacro/wheel.urdf.xacro" />
 	<link name="origin_link"/>
 	<link name="base_link">
@@ -34,26 +35,16 @@
 		<origin xyz="0 0 0.02"/>
 	</joint>
-	<xacro:rim_macro
-		name="front_left"
-		color="0.3 0 0"
-		xyz="0.053 0.05300221419 0"
-		rpy="1.570796326794896 0 -0.81">
-	<mesh scale="10 10 10"/>
-	</xacro:rim_macro>
-	<xacro:rim_macro
-		name="front_right"
-		color="0 0 0.3"
-		xyz="0.053 -0.05300221419 0"
-		rpy="1.570796326794896 0 -2.39"/>
-	<xacro:rim_macro
-		name="back_right"
-		color="0 0.3 0"
-		xyz="-0.053 -0.05300221419 0"
-		rpy="1.570796326794896 0 2.39"/>
-	<xacro:rim_macro
-		name="back_left"
-		color="0 0.2 0.2"
-		xyz="-0.053 0.05300221419 0"
-		rpy="1.570796326794896 0 0.81"/>
+	<xacro:omni_wheel wheel_prefix="front_right">
+		<origin xyz="0.053 -0.05300221419 0" rpy="1.570796326794896 0 -2.39"/>
+	</xacro:omni_wheel>
+	<xacro:omni_wheel wheel_prefix="back_right">
+		<origin xyz="-0.053 -0.05300221419 0" rpy="1.570796326794896 0 2.39"/>
+	</xacro:omni_wheel>
+	<xacro:omni_wheel wheel_prefix="back_left">
+		<origin xyz="-0.053 0.05300221419 0" rpy="1.570796326794896 0 0.81"/>
+	</xacro:omni_wheel>
+	<xacro:omni_wheel wheel_prefix="front_left">
+		<origin xyz="0.053 0.05300221419 0" rpy="1.570796326794896 0 -0.81"/>
+	</xacro:omni_wheel>
 	<joint name="scan_joint" type="fixed">
     	<parent link="base_link"/>

File: omnibase_description/xacro/wheel.urdf.xacro (robot description, xacro)
@@ -1,5 +1,5 @@
 <?xml version="1.0"?>
 <robot xmlns:xacro="http://ros.org/wiki/xacro" name="husky_wheel">
-	<xacro:macro name="husky_wheel" params="wheel_prefix *joint_pose">
+	<xacro:macro name="omni_wheel" params="wheel_prefix *joint_pose">
 		<link name="${wheel_prefix}_wheel_link">
 			<inertial>
@@ -11,5 +11,5 @@
 				<origin xyz="0 0 0" rpy="0 0 0" />
 				<geometry>
-					<cylinder length="0.05" radius="0.1" />
+					<cylinder length="0.02" radius="0.04" />
 				</geometry>
 			</visual>
@@ -17,6 +17,9 @@
 				<origin xyz="0 0 0" rpy="0 0 0" />
 				<geometry>
-					<cylinder length="0.05" radius="0.1" />
+					<cylinder length="0.02" radius="0.04" />
 				</geometry>
+				<surface>
+					<bounce restitution_coefficient="0.000001" />
+				</surface>
 			</collision>
 		</link>
@@ -27,4 +30,5 @@
 			<kd value="1.0" />
 			<fdir1 value="0 0 1"/>
+			<maxContacts value= "1"/>
 		</gazebo>
 		<joint name="${wheel_prefix}_wheel" type="continuous">
@@ -32,5 +36,5 @@
 			<child link="${wheel_prefix}_wheel_link"/>
 			<xacro:insert_block name="joint_pose"/>
-			<axis xyz="0 1 0" rpy="0 0 0" />
+			<axis xyz="0 0 1" rpy="0 0 0" />
 		</joint>
 		<transmission name="${wheel_prefix}_wheel_trans" type="SimpleTransmission">

Commit message: model update

File: omnibase_description/xacro/main.urdf.xacro (robot description, xacro)
@@ -36,14 +36,14 @@
 	</joint>
 	<xacro:omni_wheel wheel_prefix="front_right">
-		<origin xyz="0.053 -0.05300221419 0" rpy="1.570796326794896 0 -2.39"/>
+		<origin xyz="0.055 0.055 0" rpy="1.570796326794896 0 -0.78539816339"/>
+	</xacro:omni_wheel>
+	<xacro:omni_wheel wheel_prefix="front_left">
+		<origin xyz="0.055 -0.055 0" rpy="1.570796326794896 0 -2.35619449019"/>
+	</xacro:omni_wheel>
+	<xacro:omni_wheel wheel_prefix="back_left">
+		<origin xyz="-0.055 -0.055 0" rpy="1.570796326794896 0 2.35619449019"/>
 	</xacro:omni_wheel>
 	<xacro:omni_wheel wheel_prefix="back_right">
-		<origin xyz="-0.053 -0.05300221419 0" rpy="1.570796326794896 0 2.39"/>
-	</xacro:omni_wheel>
-	<xacro:omni_wheel wheel_prefix="back_left">
-		<origin xyz="-0.053 0.05300221419 0" rpy="1.570796326794896 0 0.81"/>
-	</xacro:omni_wheel>
-	<xacro:omni_wheel wheel_prefix="front_left">
-		<origin xyz="0.053 0.05300221419 0" rpy="1.570796326794896 0 -0.81"/>
+		<origin xyz="-0.055 0.055 0" rpy="1.570796326794896 0 0.78539816339"/>
 	</xacro:omni_wheel>
 	<joint name="scan_joint" type="fixed">

File: omnibase_description/xacro/wheel.urdf.xacro (robot description, xacro)
@@ -20,13 +20,13 @@
 				</geometry>
 				<surface>
-					<bounce restitution_coefficient="0.000001" />
+					<bounce restitution_coefficient="0.0001" />
 				</surface>
 			</collision>
 		</link>
 		<gazebo reference="${wheel_prefix}_wheel_link">
-			<mu1 value="0"/>
-			<mu2 value="1.0"/>
+			<mu1 value="0.2"/>
+			<mu2 value="1.5"/>
 			<kp value="10000000.0" />
-			<kd value="1.0" />
+			<kd value="10000.0" />
 			<fdir1 value="0 0 1"/>
 			<maxContacts value= "1"/>

Commit message: Fixed omniwheel size

File: omnibase_description/xacro/main.urdf.xacro (robot description, xacro)
@@ -18,5 +18,5 @@
 	<visual>
 		<geometry>
-			<mesh filename="package://omnibase_description/meshes/sq_base.stl"/>
+			<mesh filename="package://omnibase_description/meshes/trotbot_full_stl.stl" scale="0.001 0.001 0.001"/>
 		</geometry>
 		<material name="base_material">
@@ -26,5 +26,5 @@
 	<collision>
 		<geometry>
-			<mesh filename="package://omnibase_description/meshes/sq_base.stl"/>
+			<mesh filename="package://omnibase_description/meshes/trotbot_full_stl.stl" scale="0.001 0.001 0.001"/>
 		</geometry>
 	</collision>
@@ -36,14 +36,14 @@
 	</joint>
 	<xacro:omni_wheel wheel_prefix="front_right">
-		<origin xyz="0.055 0.055 0" rpy="1.570796326794896 0 -0.78539816339"/>
+		<origin xyz="0.22 0.22 0" rpy="1.570796326794896 0 -0.78539816339"/>
 	</xacro:omni_wheel>
 	<xacro:omni_wheel wheel_prefix="front_left">
-		<origin xyz="0.055 -0.055 0" rpy="1.570796326794896 0 -2.35619449019"/>
+		<origin xyz="0.22 -0.22 0" rpy="1.570796326794896 0 -2.35619449019"/>
 	</xacro:omni_wheel>
 	<xacro:omni_wheel wheel_prefix="back_left">
-		<origin xyz="-0.055 -0.055 0" rpy="1.570796326794896 0 2.35619449019"/>
+		<origin xyz="-0.22 -0.22 0" rpy="1.570796326794896 0 2.35619449019"/>
 	</xacro:omni_wheel>
 	<xacro:omni_wheel wheel_prefix="back_right">
-		<origin xyz="-0.055 0.055 0" rpy="1.570796326794896 0 0.78539816339"/>
+		<origin xyz="-0.22 0.22 0" rpy="1.570796326794896 0 0.78539816339"/>
 	</xacro:omni_wheel>
 	<joint name="scan_joint" type="fixed">
@@ -80,10 +80,4 @@
   	</joint>
   	<link name="body_link">
-  		<visual>
-  			<geometry>
-       			<mesh filename="package://omnibase_description/meshes/body.STL"/>
-      		</geometry>
-      		<material name="base_material"/>
-      	</visual>
       	<inertial>
       		<mass value="0.1" />

File: omnibase_description/xacro/main_new.urdf.xacro (robot description, xacro)
@@ -26,5 +26,5 @@
 	<collision>
 		<geometry>
-			<mesh filename="package://omnibase_description/meshes/trotbot_full_stl.stl"/>
+			<mesh filename="package://omnibase_description/meshes/trotbot_full_stl.stl" scale="0.0003 0.0003 0.0003"/>
 		</geometry>
 	</collision>

File: omnibase_description/xacro/wheel.urdf.xacro (robot description, xacro)
@@ -11,5 +11,5 @@
 				<origin xyz="0 0 0" rpy="0 0 0" />
 				<geometry>
-					<cylinder length="0.01" radius="0.01" />
+					<cylinder length="0.03" radius="0.06" />
 				</geometry>
 			</visual>
@@ -17,5 +17,5 @@
 				<origin xyz="0 0 0" rpy="0 0 0" />
 				<geometry>
-					<cylinder length="0.01" radius="0.01" />
+					<cylinder length="0.03" radius="0.06" />
 				</geometry>
 				<surface>

Commit message: changes in the model

File: omnibase_description/xacro/main.urdf.xacro (robot description, xacro)
@@ -7,5 +7,5 @@
 	<link name="base_link">
 	<inertial>
-		<mass value="0.08723"/>
+		<mass value="2"/>
 		<inertia
 			ixx="0.0100"
@@ -47,5 +47,5 @@
     	<parent link="base_link"/>
     	<child link="base_scan"/>
-    	<origin xyz="-0.005 0 0.064" rpy="0 0 0"/>
+    	<origin xyz="-0.005 0 0.235" rpy="0 0 0"/>
   	</joint>
 	<link name="base_scan">
@@ -53,5 +53,5 @@
     	<origin xyz="0 0 0.0" rpy="0 0 0"/>
     	<geometry>
-       		<mesh filename="package://omnibase_description/meshes/lds.stl" scale="0.0003 0.0003 0.0003"/>
+       		<mesh filename="package://omnibase_description/meshes/lds.stl" scale="0.00085 0.00085 0.00085"/>
       	</geometry>
       	<material name="dark"/>

Commit message: Realsense D435 added to model

File: omnibase_description/xacro/main.urdf.xacro (robot description, xacro)
@@ -4,4 +4,5 @@
 	<xacro:include filename="$(find omnibase_description)/xacro/gazebo.urdf.xacro"/>
 	<xacro:include filename="$(find omnibase_description)/xacro/wheel.urdf.xacro" />
+	<xacro:include filename="$(find omnibase_description)/xacro/intel_realsense.urdf.xacro" />
 	<link name="origin_link"/>
 	<link name="base_link">
@@ -71,4 +72,11 @@
     </inertial>
   	</link>
+	<link name="base_cam"/>
+	<joint name="cam_joint" type="fixed">
+		<origin xyz="0.06 0 0.22" rpy="0 0 0" />
+		<parent link="base_link"/>
+		<child link="base_cam" />
+	</joint>
+	<xacro:intel_realsense_mount prefix="omnibase" topic="realsense" parent_link="base_cam"/>
   	<joint name="body_joint" type="fixed">
   		<parent link="base_link"/>
