Commit message: minor changes in the model

File: omnibase_description/xacro/intel_realsense.urdf.xacro (robot description, xacro)
@@ -78,5 +78,5 @@
         <geometry>
           <!-- Origin of this mesh is the base of the bracket. -->
-          <mesh filename="package://omnibase_description/meshes/d415.stl" />
+          <mesh filename="package://omnibase_description/meshes/d415.stl" scale="0.8 0.8 0.8"/>
         </geometry>
         <material name="white" />

File: omnibase_description/xacro/main_new.urdf.xacro (robot description, xacro)
@@ -56,5 +56,5 @@
     	<origin xyz="0 0 0.0" rpy="0 0 0"/>
     	<geometry>
-       		<mesh filename="package://omnibase_description/meshes/lds.stl" scale="0.0003 0.0003 0.0003"/>
+       		<mesh filename="package://omnibase_description/meshes/lds.stl" scale="0.0008 0.0008 0.0008"/>
       	</geometry>
       	<material name="dark"/>

File: omnibase_description/xacro/main_realsense.urdf.xacro (robot description, xacro)
@@ -54,5 +54,5 @@
     	<origin xyz="0 0 0.0" rpy="0 0 0"/>
     	<geometry>
-       		<mesh filename="package://omnibase_description/meshes/lds.stl" scale="0.00085 0.00085 0.00085"/>
+       		<mesh filename="package://omnibase_description/meshes/lds.stl" scale="0.0008 0.0008 0.0008"/>
       	</geometry>
       	<material name="dark"/>
@@ -74,5 +74,5 @@
 	<link name="base_cam"/>
 	<joint name="cam_joint" type="fixed">
-		<origin xyz="0.06 0 0.22" rpy="0 0 0" />
+		<origin xyz="0.06 0 0.21" rpy="0 0 0" />
 		<parent link="base_link"/>
 		<child link="base_cam" />
